Commit message: v3

File: src/youbot_description/urdf/youbot.urdf (robot description, URDF)
Before this commit: robot youbot, 22 links, 21 joints
Links:
- added link color_cam
- added link depth_cam
- added link gripper_tcp
- added link stand
- link plate_link: geometry collision mesh filename=package://youbot_description/meshes/youbot_plate/plate.dae; visual mesh filename=package://youbot_description/meshes/youbot_plate/plate.dae
Joints:
- added joint color_cam_joint: type fixed, parent stand, child color_cam, origin xyz=-0.06673 0.04023 0.13603 rpy=-2.0944 0 -0.785398, axis 0 0 0
- added joint depth_cam_joint: type fixed, parent stand, child depth_cam, origin xyz=-0.05613 0.02962 0.13603 rpy=-2.0944 0 -0.785398, axis 0 0 0
- added joint gripper_tcp_joint: type fixed, parent arm_link_5, child gripper_tcp, origin xyz=0 0 0.075 rpy=0 0 0
- added joint stand_joint: type fixed, parent plate_link, child stand, origin xyz=0.06 0.06 -0.001, axis 0 0 0

Commit message: v5

File: src/youbot_description/urdf/youbot.urdf (robot description, URDF)
Before this commit: robot youbot, 26 links, 25 joints
Joints:
- joint wheel_joint_bl: type continuous -> fixed
- joint wheel_joint_br: type continuous -> fixed
- joint wheel_joint_fl: type continuous -> fixed
- joint wheel_joint_fr: type continuous -> fixed
- joint world_joint: type continuous -> fixed
